File: KiCAD/22257_DevBoard/22257_DevBoard/22257_DevBoard.kicad_pcb (KiCad board)
At the start: 6 copper layers, 90 parts, among them J1 TD-120-G-AACON40_2X20_TU_HTS_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, J2 TD-120-G-AACON40_2X20_TU_HTS_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, J3 Screw_Terminal_01x02, J4 Conn_Coaxial, J5 Conn_Coaxial, J6 Conn_Coaxial, J7 Conn_Coaxial, U10 74LVC1G17, U11 74LVC1G17, U3 TPS73633DBV, U4 TPS562202, U5 INA219AxD, U6 INA219AxD, U7 BME680, U8 74LVC1G17, U9 74LVC1G17

Commit message: EOD
Connections:
- J1 pad 28: BRD_PPS_IN -> /MicroZed_Headers/35_D18
- J1 pad 5: /MicroZed_Headers/35_J16 -> BRD_10MHz_OUT
- J2 pad 31: BRD_10MHz_OUT -> /MicroZed_Headers/34_V18
- JX1 pad 25: BRD_PPS_IN -> /MicroZed_Headers/35_D18
- JX1 pad 90: /MicroZed_Headers/35_J16 -> BRD_10MHz_OUT
- JX2 pad 75: BRD_10MHz_OUT -> /MicroZed_Headers/34_V18
Routing:
- net BRD_10MHz_OUT: track 24.3 -> 181.1 mm, vias 0 -> 1
- net BRD_PPS_IN: track 36.4 -> 14.2 mm, vias 1 -> 0
- net /MicroZed_Headers/35_D18: track 0.00 -> 22.2 mm, vias 0 -> 1
- net /MicroZed_Headers/34_V18: track 0.00 -> 15.5 mm
- net /MicroZed_Headers/35_J16: track 12.4 -> 0.00 mm
- net CSAC_Tx: track 109.0 -> 99.6 mm
- net CSAC_PPS_OUT: track 121.9 -> 113.2 mm
- net PM_SCL_5V: track 36.3 -> 30.0 mm, vias 2 -> 1
- net CSAC_BITE: track 84.7 -> 89.8 mm, vias 1 -> 0
- net ES_CSB: track 174.0 -> 172.4 mm
- net CSAC_PPS_IN: track 158.4 -> 157.3 mm
- net ES_SCK: track 140.4 -> 139.4 mm

Commit message: Power Pours
Parts:
- moved TP16 30.8 mm to (169.7, 2.32), turned to 90 degrees
- moved TP15 23.8 mm to (170.0, 6.63), turned to 90 degrees
- moved L2 17.8 mm to (167.5, 20.5), turned to -90 degrees
- moved U5 17.7 mm to (162.6, 7.82), turned to 180 degrees
- moved C7 17.5 mm to (140.6, 5.03)
- moved C8 17.5 mm to (142.7, 5.03)
- moved C16 16.6 mm to (161.4, 4.12), turned to 0 degrees
- moved U3 16.4 mm to (137.4, 5.08)
- moved C5 16.4 mm to (134.2, 4.16)
- moved C9 16.4 mm to (138.0, 1.49)
- moved C12 16.4 mm to (173.7, 22.8), turned to -90 degrees
- moved TP18 16.4 mm to (126.7, 9.91)
- moved C11 15.9 mm to (175.5, 22.9), turned to -90 degrees
- moved R1 15.4 mm to (140.6, 2.28), turned to 180 degrees
- moved TP17 12.5 mm to (131.3, 9.91)
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Connections:
- C11 pad 2: Net-(C11-Pad2) -> Net-(U5-IN+)
- C12 pad 2: Net-(C11-Pad2) -> Net-(U5-IN+)
- L2 pad 2: Net-(C11-Pad2) -> Net-(U5-IN+)
- R4 pad 2: Net-(C11-Pad2) -> Net-(U5-IN+)
- R6 pad 2: Net-(U5-IN-) -> Net-(U5-IN+)
- R7 pad 2: Net-(U6-IN-) -> Net-(U3-OUT)
- TP10 pad 1: Net-(C11-Pad2) -> Net-(U5-IN+)
- U5 pad 7: Net-(U5-IN-) -> +5V
- U6 pad 7: Net-(U6-IN-) -> +3.3V
- U6 pad 8: Net-(U6-IN+) -> Net-(U3-OUT)
Routing:
- net BRD_PPS_IN: track 14.2 -> 195.5 mm, vias 0 -> 2
- net BRD_PPS_OUT: track 0.00 -> 155.6 mm, vias 0 -> 1
- net PM_SCL_3v3: track 113.4 -> 94.1 mm
- net PM_SDA_3v3: track 111.9 -> 95.8 mm
- net Net-(U4-EN): track 0.00 -> 6.98 mm
- net +3.3V: track 0.00 -> 4.02 mm, vias 0 -> 4
- net Net-(U3-EN): track 0.00 -> 3.85 mm
- net +5V: track 0.00 -> 3.80 mm
- net +12V: track 0.00 -> 3.78 mm
- net PM_SCL_5V: track 30.0 -> 26.5 mm
- net Net-(U3-NR): track 0.00 -> 2.34 mm
- net CSAC_BITE: track 89.8 -> 92.0 mm
- net CSAC_RF_OUT: track 114.3 -> 116.5 mm
- net PM_SDA_5V: track 27.5 -> 25.5 mm, vias 2 -> 1
- net CSAC_PPS_OUT: track 113.2 -> 114.6 mm
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- added copper zone on F.Cu, net +12V
- added copper zone on In4.Cu, net +12V
- added copper zone on F.Cu, net +3.3V
- added copper zone on In4.Cu, net +3.3V
- added copper zone on In4.Cu, net +5V
- added copper zone on B.Cu, net GND
- added copper zone on F.Cu, net GND
- added copper zone on F.Cu, net Net-(U3-IN)
- added copper zone on F.Cu, net Net-(U3-OUT)
- added copper zone on F.Cu, net Net-(U4-SW)
- added copper zone on F.Cu, net Net-(U5-IN+)
Other:
- board outline added: 213.1 x 99.1 mm

Commit message: EOD
Nearly finished routing
Parts:
- added C23: 47u, Capacitor_SMD:C_0603_1608Metric, F.Cu at (89.1, 23.9)
- added C24: 47u, Capacitor_SMD:C_0603_1608Metric, F.Cu at (97.8, 64.4)
- moved C1 2.80 mm to (152.1, 39.9)
- moved C2 2.58 mm to (154.4, 39.9)
- moved C3 2.21 mm to (176.3, 81.0)
- moved C4 1.14 mm to (174.2, 81.0)
Connections:
- J1 pad 3: 5V -> +5V
- J1 pad 37: 5V -> +5V
- J1 pad 38: 5V -> +5V
- J1 pad 4: 5V -> +5V
- J2 pad 1: 5V -> +5V
- J2 pad 2: 5V -> +5V
- J2 pad 3: 5V -> +5V
- J2 pad 37: 5V -> +5V
- J2 pad 38: 5V -> +5V
- J2 pad 4: 5V -> +5V
- JX1 pad 10: 3V3 -> +3.3V
- JX1 pad 11: 3V3 -> +3.3V
- JX1 pad 12: 5V -> +5V
- JX1 pad 57: 5V -> +5V
- JX1 pad 58: 5V -> +5V
- JX1 pad 59: 5V -> +5V
- JX1 pad 60: 5V -> +5V
- JX1 pad 78: 3V3 -> +3.3V
- JX1 pad 79: 3V3 -> +3.3V
- JX1 pad 80: 3V3 -> +3.3V
- JX1 pad 98: 3V3 -> +3.3V
- JX2 pad 5: 5V -> +5V
- JX2 pad 57: 5V -> +5V
- JX2 pad 58: 5V -> +5V
- JX2 pad 59: 5V -> +5V
- JX2 pad 60: 5V -> +5V
- JX2 pad 78: 3V3 -> +3.3V
- JX2 pad 79: 3V3 -> +3.3V
- JX2 pad 80: 3V3 -> +3.3V
Routing:
- net +5V: track 3.80 -> 54.0 mm, vias 0 -> 18
- net +3.3V: track 4.02 -> 15.2 mm, vias 4 -> 23
- net ES_SDO: track 136.4 -> 134.7 mm

Commit message: Routing progress
Parts:
- moved TP17 0.07 mm to (131.3, 9.86)
Routing:
- net PM_SDA_5V: track 25.5 -> 161.2 mm, vias 1 -> 3
- net PM_SCL_5V: track 26.5 -> 157.1 mm, vias 1 -> 3
- net CSAC_Tune: track 24.5 -> 116.6 mm
- net +3.3V: track 15.2 -> 95.2 mm, vias 23 -> 42
- net Net-(U5-IN+): track 0.07 -> 13.7 mm, vias 0 -> 2
- net Net-(U6-A0): track 0.00 -> 6.62 mm
- net ES_CSB: track 172.4 -> 166.1 mm
- net Net-(U6-A1): track 0.00 -> 5.79 mm
- net ES_SDI: track 147.9 -> 143.2 mm
- net CSAC_BITE: track 92.0 -> 96.2 mm
- net BRD_PPS_OUT: track 155.6 -> 159.3 mm
- net ES_SCK: track 139.4 -> 136.6 mm
- net CSAC_RF_OUT: track 116.5 -> 119.1 mm
- net TST_01: track 105.4 -> 102.9 mm
- net TCXO_A0: track 113.6 -> 111.2 mm
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