File: KiCAD/22257_DevBoard/22257_DevBoard/power-connectors.kicad_sch (KiCad schematic)
At the start: 49 parts, among them J3 Screw_Terminal_01x02, J4 Conn_Coaxial, J5 Conn_Coaxial, J6 Conn_Coaxial, J7 Conn_Coaxial, U3 TPS73633DBV, U4 TPS562202, U5 INA219AxD, U6 INA219AxD

Commit message: Started layout
Parts:
- H1, H2, H3, H4: footprint ZED_BREAKOUT_v22:5,0-PAD -> MountingHole:MountingHole_3.2mm_M3
- R13, R8: footprint (none) -> Resistor_SMD:R_0603_1608Metric
- R6, R7: footprint (none) -> 2222_DevBoar_Footprints:BVT-I-R0002-1
- TP1, TP2, TP3: footprint (none) -> TestPoint:TestPoint_THTPad_2.5x2.5mm_Drill1.2mm
- TP10, TP4, TP5, TP6, TP7, TP8, TP9: footprint (none) -> TestPoint:TestPoint_2Pads_Pitch5.08mm_Drill1.3mm
Changed lines of the file:
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@@
 			)
 		)
-		(property "Footprint" ""
+		(property "Footprint" "TestPoint:TestPoint_2Pads_Pitch5.08mm_Drill1.3mm"
 			(at 143.51 219.71 0)
 			(effects
@@
 			)
 		)
-		(property "Footprint" ""
+		(property "Footprint" "2222_DevBoar_Footprints:BVT-I-R0002-1"
 			(at 144.78 117.602 90)
 			(effects
@@
 			)
 		)
-		(property "Footprint" ""
+		(property "Footprint" "TestPoint:TestPoint_2Pads_Pitch5.08mm_Drill1.3mm"
 			(at 144.78 109.22 0)
 			(effects
@@
 			)
 		)
-		(property "Footprint" "ZED_BREAKOUT_v22:5,0-PAD"
+		(property "Footprint" "MountingHole:MountingHole_3.2mm_M3"
 			(at 271.78 246.38 0)
 			(effects
@@
 			)
 		)
-		(property "Footprint" "ZED_BREAKOUT_v22:5,0-PAD"
+		(property "Footprint" "MountingHole:MountingHole_3.2mm_M3"
 			(at 238.76 246.38 0)
 			(effects
@@
 			)
 		)
-		(property "Footprint" ""
+		(property "Footprint" "TestPoint:TestPoint_2Pads_Pitch5.08mm_Drill1.3mm"
 			(at 143.51 245.11 0)
 			(effects
@@
 			)
 		)
-		(property "Footprint" "ZED_BREAKOUT_v22:5,0-PAD"
+		(property "Footprint" "MountingHole:MountingHole_3.2mm_M3"
 			(at 250.19 246.38 0)
 			(effects
@@
 			)
 		)
-		(property "Footprint" ""
+		(property "Footprint" "TestPoint:TestPoint_THTPad_2.5x2.5mm_Drill1.2mm"
 			(at 176.53 30.48 0)
 			(effects
@@
 			)
 		)
-		(property "Footprint" ""
+		(property "Footprint" "TestPoint:TestPoint_2Pads_Pitch5.08mm_Drill1.3mm"
 			(at 68.58 246.38 0)
 			(effects
@@
 			)
 		)
-		(property "Footprint" ""
+		(property "Footprint" "TestPoint:TestPoint_THTPad_2.5x2.5mm_Drill1.2mm"
 			(at 46.99 41.91 0)
 			(effects
@@
 			)
 		)
-		(property "Footprint" ""
+		(property "Footprint" "2222_DevBoar_Footprints:BVT-I-R0002-1"
 			(at 157.48 42.672 90)
 			(effects
@@
 			)
 		)
-		(property "Footprint" ""
+		(property "Footprint" "TestPoint:TestPoint_THTPad_2.5x2.5mm_Drill1.2mm"
 			(at 165.1 110.49 0)
 			(effects
@@
 			)
 		)
-		(property "Footprint" ""
+		(property "Footprint" "TestPoint:TestPoint_2Pads_Pitch5.08mm_Drill1.3mm"
 			(at 68.58 220.98 0)
 			(effects
@@
 			)
 		)
-		(property "Footprint" "ZED_BREAKOUT_v22:5,0-PAD"
+		(property "Footprint" "MountingHole:MountingHole_3.2mm_M3"
 			(at 261.62 246.38 0)
 			(effects
@@
 			)
 		)
-		(property "Footprint" ""
+		(property "Footprint" "Resistor_SMD:R_0603_1608Metric"
 			(at 270.764 48.006 90)
 			(effects
@@
 			)
 		)
-		(property "Footprint" ""
+		(property "Footprint" "Resistor_SMD:R_0603_1608Metric"
 			(at 236.474 48.006 90)
 			(effects
@@
 			)
 		)
-		(property "Footprint" ""
+		(property "Footprint" "TestPoint:TestPoint_2Pads_Pitch5.08mm_Drill1.3mm"
 			(at 157.48 34.29 0)
 			(effects
@@
 			)
 		)
-		(property "Footprint" ""
+		(property "Footprint" "TestPoint:TestPoint_2Pads_Pitch5.08mm_Drill1.3mm"
 			(at 73.66 184.15 0)
 			(effects

Commit message: Finished Component Placement and Arrangement.
Parts:
- removed H1, H2, H3, H4: MOUNT-PAD-ROUND5.0, MountingHole:MountingHole_3.2mm_M3, symbol ZED_BREAKOUT_v22-eagle-import:MOUNT-PAD-ROUND5.0
- added H1, H10, H11, H2, H3, H4, H8, H9: MountingHole_Pad, MountingHole:MountingHole_3.2mm_M3_Pad, symbol Mechanical:MountingHole_Pad
- added TP11, TP12, TP13, TP14, TP15, TP16, TP17, TP18: TestPoint, TestPoint:TestPoint_THTPad_2.5x2.5mm_Drill1.2mm, symbol Connector:TestPoint
- L1, L2: footprint (none) -> Inductor_SMD:L_Bourns-SRU8043
Connections:
- net GND: now also H1.1, H10.1, H11.1, H2.1, H3.1, H4.1, H8.1, H9.1, TP11.1, TP12.1, TP13.1, TP14.1
- net at U6.1 (A1): now also TP17.1
- net at U6.2 (A0): now also TP18.1
- net at U5.1 (A1): now also TP15.1
- net at U5.2 (A0): now also TP16.1

Commit message: Power Pours
Parts:
- R6, R7: symbol Device:R_Shunt_US -> Device:R
Connections:
- net +3.3V: now also U6.7 (IN-)
- net +5V: now also U5.7 (IN-)
- net at R7.2: now also C6.1, TP9.1, U3.5 (OUT), U6.8 (IN+); no longer U6.7 (IN-)
- net at C11.2, C12.2, L2.2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: now also R6.2, U5.8 (IN+); no longer R6.4
Changed lines of the file:
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@@
 	)
 	(junction
+		(at 152.4 44.45)
+		(diameter 0)
+		(color 0 0 0 0)
+	)
+	(junction
 		(at 231.14 243.84)
 		(diameter 0)
@@
 	)
 	(junction
+		(at 149.86 119.38)
+		(diameter 0)
+		(color 0 0 0 0)
+	)
+	(junction
 		(at 156.21 109.22)
 		(diameter 0)
@@
 	)
 	(junction
+		(at 139.7 119.38)
+		(diameter 0)
+		(color 0 0 0 0)
+	)
+	(junction
 		(at 45.72 62.23)
 		(diameter 0)
@@
 	)
 	(junction
+		(at 162.56 44.45)
+		(diameter 0)
+		(color 0 0 0 0)
+	)
+	(junction
 		(at 77.47 237.49)
 		(diameter 0)
@@
 	(wire
 		(pts
+			(xy 139.7 119.38) (xy 140.97 119.38)
+		)
+		(stroke
+			(width 0)
+			(type default)
+		)
+	)
+	(wire
+		(pts
 			(xy 107.95 48.26) (xy 105.41 48.26)
 		)
@@
 	(wire
 		(pts
+			(xy 149.86 123.19) (xy 149.86 119.38)
+		)
+		(stroke
+			(width 0)
+			(type default)
+		)
+	)
+	(wire
+		(pts
 			(xy 231.14 270.51) (xy 231.14 274.32)
 		)
@@
 	(wire
 		(pts
+			(xy 152.4 44.45) (xy 153.67 44.45)
+		)
+		(stroke
+			(width 0)
+			(type default)
+		)
+	)
+	(wire
+		(pts
 			(xy 90.17 130.81) (xy 90.17 133.35)
 		)
@@
 	(wire
 		(pts
+			(xy 152.4 48.26) (xy 152.4 44.45)
+		)
+		(stroke
+			(width 0)
+			(type default)
+		)
+	)
+	(wire
+		(pts
 			(xy 166.37 34.29) (xy 166.37 29.21)
 		)
@@
 	(wire
 		(pts
+			(xy 142.24 123.19) (xy 139.7 123.19)
+		)
+		(stroke
+			(width 0)
+			(type default)
+		)
+	)
+	(wire
+		(pts
 			(xy 148.59 219.71) (xy 156.21 219.71)
 		)
@@
 	(wire
 		(pts
-			(xy 160.02 48.26) (xy 160.02 57.15)
+			(xy 160.02 46.99) (xy 160.02 57.15)
 		)
 		(stroke
@@
 	(wire
 		(pts
+			(xy 154.94 48.26) (xy 152.4 48.26)
+		)
+		(stroke
+			(width 0)
+			(type default)
+		)
+	)
+	(wire
+		(pts
 			(xy 95.25 52.07) (xy 97.79 52.07)
 		)
@@
 	(wire
 		(pts
+			(xy 148.59 119.38) (xy 149.86 119.38)
+		)
+		(stroke
+			(width 0)
+			(type default)
+		)
+	)
+	(wire
+		(pts
 			(xy 226.06 270.51) (xy 231.14 270.51)
 		)
@@
 	(wire
 		(pts
+			(xy 139.7 123.19) (xy 139.7 119.38)
+		)
+		(stroke
+			(width 0)
+			(type default)
+		)
+	)
+	(wire
+		(pts
+			(xy 147.32 123.19) (xy 149.86 123.19)
+		)
+		(stroke
+			(width 0)
+			(type default)
+		)
+	)
+	(wire
+		(pts
 			(xy 237.49 36.83) (xy 237.49 44.45)
 		)
@@
 	(wire
 		(pts
+			(xy 162.56 46.99) (xy 162.56 44.45)
+		)
+		(stroke
+			(width 0)
+			(type default)
+		)
+	)
+	(wire
+		(pts
 			(xy 115.57 121.92) (xy 119.38 121.92)
 		)
@@
 	(wire
 		(pts
+			(xy 161.29 44.45) (xy 162.56 44.45)
+		)
+		(stroke
+			(width 0)
+			(type default)
+		)
+	)
+	(wire
+		(pts
 			(xy 45.72 62.23) (xy 45.72 66.04)
 		)
@@
 	(wire
 		(pts
+			(xy 160.02 46.99) (xy 162.56 46.99)
+		)
+		(stroke
+			(width 0)
+			(type default)
+		)
+	)
+	(wire
+		(pts
 			(xy 129.54 237.49) (xy 134.62 237.49)
 		)
@@
 	)
 	(symbol
-		(lib_id "Device:R_Shunt_US")
+		(lib_id "Device:R")
 		(at 144.78 119.38 270)
 		(unit 1)
@@
 			)
 		)
-		(property "Description" "Shunt resistor, US symbol"
+		(property "Description" "Resistor"
 			(at 144.78 119.38 0)
 			(effects
@@
 		(pin "1"
 		)
-		(pin "3"
-		)
-		(pin "4"
-		)
 		(pin "2"
 		)
@@
 	)
 	(symbol
-		(lib_id "Device:R_Shunt_US")
+		(lib_id "Device:R")
 		(at 157.48 44.45 270)
 		(unit 1)
@@
 			)
 		)
-		(property "Description" "Shunt resistor, US symbol"
+		(property "Description" "Resistor"
 			(at 157.48 44.45 0)
 			(effects
@@
 		(pin "1"
 		)
-		(pin "3"
-		)
-		(pin "4"
-		)
 		(pin "2"

Commit message: EOD
Nearly finished routing
Parts:
- added C23, C24: 47u, Capacitor_SMD:C_0603_1608Metric, symbol Device:C
Connections:
- net +3.3V: now also C23.2, C24.2
- net GND: now also C23.1, C24.1

Commit message: DONE ROUTINGgit add .git add .
Parts:
- added C25: 47u, Capacitor_SMD:C_0603_1608Metric, symbol Device:C
Connections:
- net +5V: now also C25.2
- net GND: now also C25.1
Other:
- moved on the sheet: C23, C24
