File: KiCAD/22257_DevBoard/22257_DevBoard/power-connectors.kicad_sch (KiCad schematic)
At the start: 64 parts, among them J3 Screw_Terminal_01x02, J4 Conn_Coaxial, J5 Conn_Coaxial, J6 Conn_Coaxial, J7 Conn_Coaxial, U3 TPS73633DBV, U4 TPS562202, U5 INA219AxD, U6 INA219AxD

Commit message: Done :D
Existence is pain
Parts:
- R6, R7: value R_Shunt_US -> 2m
Other:
- note added: "Current Resolution = 5mA"
Changed lines of the file:
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@@
 		)
 	)
+	(text "Current Resolution = 5mA"
+		(exclude_from_sim no)
+		(at 167.386 66.294 0)
+		(effects
+			(font
+				(size 1.27 1.27)
+			)
+		)
+	)
 	(text "Power Monitor"
 		(exclude_from_sim no)
@@
 			)
 		)
-		(property "Value" "R_Shunt_US"
+		(property "Value" "2m"
 			(at 144.78 115.57 90)
 			(effects
@@
 			)
 		)
-		(property "Value" "R_Shunt_US"
+		(property "Value" "2m"
 			(at 157.48 40.64 90)
 			(effects

Commit message: Added notes from review with Carlos
Other:
- note added: "Bulk Capacitances"
- note added: "HARDWIRE ADDRESS"
- moved on the sheet: C23, C24, C25, D1, D2, D7, R13, R2, R8, TP11, TP12, TP13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

Commit message: Started BOM
Parts:
- removed TP15, TP16, TP17, TP18: TestPoint, TestPoint:TestPoint_THTPad_2.5x2.5mm_Drill1.2mm, symbol Connector:TestPoint
Connections:
- net +5V: now also U5.1 (A1), U5.2 (A0)
- net GND: now also U6.1 (A1), U6.2 (A0)
Other:
- note removed: "HARDWIRE ADDRESS"

Commit message: Output Files Generated
Parts:
- C14: value .1u -> 0.1u
Changed lines of the file:
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@@
 			)
 		)
-		(property "Value" ".1u"
+		(property "Value" "0.1u"
 			(at 55.88 55.8799 0)
 			(effects
