File: KiCAD/22257_DevBoard/22257_DevBoard/oscillators.kicad_sch (KiCad schematic)
At the start: 25 parts, among them U10 74LVC1G17, U11 74LVC1G17, U7 BME680, U8 74LVC1G17, U9 74LVC1G17

Commit message: Started BOM
Connections:
- net ES_SDO is gone; now on net GND: U7.5 (SDO)
- net TCXO_A0: no longer names the net of U2.5 (A0)
- no-connect marks 0 -> 1
Changed lines of the file:
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@@
 		(color 0 0 0 0)
 	)
+	(no_connect
+		(at 280.67 59.69)
+	)
 	(wire
 		(pts
@@
 	(wire
 		(pts
-			(xy 114.3 151.13) (xy 119.38 151.13)
+			(xy 114.3 151.13) (xy 134.62 151.13)
 		)
 		(stroke
@@
 	(wire
 		(pts
+			(xy 134.62 151.13) (xy 134.62 154.94)
+		)
+		(stroke
+			(width 0)
+			(type default)
+		)
+	)
+	(wire
+		(pts
 			(xy 245.11 62.23) (xy 257.81 62.23)
 		)
@@
 		)
 	)
-	(global_label "ES_SDO"
-		(shape bidirectional)
-		(at 119.38 151.13 0)
-		(fields_autoplaced yes)
-		(effects
-			(font
-				(size 1.27 1.27)
-			)
-			(justify left)
-		)
-		(property "Intersheetrefs" "${INTERSHEET_REFS}"
-			(at 130.6126 151.13 0)
-			(effects
-				(font
-					(size 1.27 1.27)
-				)
-				(justify left)
-				(hide yes)
-			)
-		)
-	)
 	(global_label "ES_CSB"
 		(shape input)
@@
 		)
 	)
-	(global_label "TCXO_A0"
-		(shape input)
-		(at 280.67 59.69 180)
-		(fields_autoplaced yes)
-		(effects
-			(font
-				(size 1.27 1.27)
-			)
-			(justify right)
-		)
-		(property "Intersheetrefs" "${INTERSHEET_REFS}"
-			(at 269.6415 59.69 0)
-			(effects
-				(font
-					(size 1.27 1.27)
-				)
-				(justify right)
-				(hide yes)
-			)
-		)
-	)
 	(global_label "TST_01"
 		(shape input)
@@
 					(unit 1)
 				)
+			)
+		)
+	)
+	(symbol
+		(lib_id "power:GND")
+		(at 134.62 154.94 0)
+		(unit 1)
+		(exclude_from_sim no)
+		(in_bom yes)
+		(on_board yes)
+		(dnp no)
+		(fields_autoplaced yes)
+		(property "Reference" "#PWR050"
+			(at 134.62 161.29 0)
+			(effects
+				(font
+					(size 1.27 1.27)
+				)
+				(hide yes)
+			)
+		)
+		(property "Value" "GND"
+			(at 134.62 160.02 0)
+			(effects
+				(font
+					(size 1.27 1.27)
+				)
+			)
+		)
+		(property "Footprint" ""
+			(at 134.62 154.94 0)
+			(effects
+				(font
+					(size 1.27 1.27)
+				)
+				(hide yes)
+			)
+		)
+		(property "Datasheet" ""
+			(at 134.62 154.94 0)
+			(effects
+				(font
+					(size 1.27 1.27)
+				)
+				(hide yes)
+			)
+		)
+		(property "Description" "Power symbol creates a global label with name \"GND\" , ground"
+			(at 134.62 154.94 0)
+			(effects
+				(font
+					(size 1.27 1.27)
+				)
+				(hide yes)
+			)
+		)
+		(pin "1"
+		)
+		(instances
+			(project "22257_DevBoard"
+				(path "/271303ce-366a-4ce1-87f0-a9575f73ea97/f8a3ba62-8e39-4a66-bf12-691136caf958"
+					(reference "#PWR050")
+					(unit 1)
+				)
